Commit message: use simpler collision shapes which are inflated by 2 mm

File: xarm_description/urdf/xarm7/xarm7.urdf.xacro (robot description, xacro)
@@ -23,5 +23,5 @@
     <xacro:unless value="${model_num >= 1305 and model_num != 1380}">
       <xacro:property name="visual_dir" value="xarm7/visual"/>
-      <xacro:property name="collision_dir" value="xarm7/visual"/>
+      <xacro:property name="collision_dir" value="xarm7/collision"/>
       <xacro:property name="add_mesh_suffix" value="true"/>
       <xacro:property name="collison_mesh_suffix" value="stl"/>
