Commit message: add mesh scale to link collision shapes; may revert later

File: xarm_description/urdf/common/common.link.xacro (robot description, xacro)
@@ -43,16 +43,16 @@
     </visual>
   </xacro:macro>
-  <xacro:macro name="common_link_collision" params="mesh_filename add_mesh_suffix:=true origin_xyz:='0 0 0' origin_rpy:='0 0 0' other_mesh_suffix:=''">
+  <xacro:macro name="common_link_collision" params="mesh_filename add_mesh_suffix:=true origin_xyz:='0 0 0' origin_rpy:='0 0 0' other_mesh_suffix:='' mesh_scale:='1.0'">
     <collision>
       <geometry>
         <xacro:if value="${add_mesh_suffix}">
-          <mesh filename="${mesh_path}/${mesh_filename}.${mesh_suffix}"/>
+          <mesh filename="${mesh_path}/${mesh_filename}.${mesh_suffix}" scale="${mesh_scale} ${mesh_scale} ${mesh_scale}"/>
         </xacro:if>
         <xacro:unless value="${add_mesh_suffix}">
           <xacro:if value="${other_mesh_suffix != ''}">
-            <mesh filename="${mesh_path}/${mesh_filename}.${other_mesh_suffix}"/>
+            <mesh filename="${mesh_path}/${mesh_filename}.${other_mesh_suffix}" scale="${mesh_scale} ${mesh_scale} ${mesh_scale}"/>
           </xacro:if>
           <xacro:unless value="${other_mesh_suffix != ''}">
-            <mesh filename="${mesh_path}/${mesh_filename}"/>
+            <mesh filename="${mesh_path}/${mesh_filename}" scale="${mesh_scale} ${mesh_scale} ${mesh_scale}"/>
           </xacro:unless>
         </xacro:unless>

File: xarm_description/urdf/xarm7/xarm7.urdf.xacro (robot description, xacro)
@@ -10,6 +10,8 @@
     joint7_lower_limit:=${-2.0*pi}  joint7_upper_limit:=${2.0*pi}
     model_num:=0
-    inertial_params_filename:='' kinematics_params_filename:='' "
+    inertial_params_filename:='' kinematics_params_filename:=''
+    collision_mesh_scale:=1.0"
     >
+    <!-- set collision_mesh_scale to 1.002 after meshes are reduced -->
     <!-- define property -->
     <xacro:if value="${model_num >= 1305 and model_num != 1380}">

Commit message: Revert "add mesh scale to link collision shapes; may revert later"
This reverts commit f0b9e785c065aa6d12f7549e2d507b5529b847d9.

File: xarm_description/urdf/common/common.link.xacro (robot description, xacro)
@@ -43,16 +43,16 @@
     </visual>
   </xacro:macro>
-  <xacro:macro name="common_link_collision" params="mesh_filename add_mesh_suffix:=true origin_xyz:='0 0 0' origin_rpy:='0 0 0' other_mesh_suffix:='' mesh_scale:='1.0'">
+  <xacro:macro name="common_link_collision" params="mesh_filename add_mesh_suffix:=true origin_xyz:='0 0 0' origin_rpy:='0 0 0' other_mesh_suffix:=''">
     <collision>
       <geometry>
         <xacro:if value="${add_mesh_suffix}">
-          <mesh filename="${mesh_path}/${mesh_filename}.${mesh_suffix}" scale="${mesh_scale} ${mesh_scale} ${mesh_scale}"/>
+          <mesh filename="${mesh_path}/${mesh_filename}.${mesh_suffix}"/>
         </xacro:if>
         <xacro:unless value="${add_mesh_suffix}">
           <xacro:if value="${other_mesh_suffix != ''}">
-            <mesh filename="${mesh_path}/${mesh_filename}.${other_mesh_suffix}" scale="${mesh_scale} ${mesh_scale} ${mesh_scale}"/>
+            <mesh filename="${mesh_path}/${mesh_filename}.${other_mesh_suffix}"/>
           </xacro:if>
           <xacro:unless value="${other_mesh_suffix != ''}">
-            <mesh filename="${mesh_path}/${mesh_filename}" scale="${mesh_scale} ${mesh_scale} ${mesh_scale}"/>
+            <mesh filename="${mesh_path}/${mesh_filename}"/>
           </xacro:unless>
         </xacro:unless>

File: xarm_description/urdf/xarm7/xarm7.urdf.xacro (robot description, xacro)
@@ -10,8 +10,6 @@
     joint7_lower_limit:=${-2.0*pi}  joint7_upper_limit:=${2.0*pi}
     model_num:=0
-    inertial_params_filename:='' kinematics_params_filename:=''
-    collision_mesh_scale:=1.0"
+    inertial_params_filename:='' kinematics_params_filename:='' "
     >
-    <!-- set collision_mesh_scale to 1.002 after meshes are reduced -->
     <!-- define property -->
     <xacro:if value="${model_num >= 1305 and model_num != 1380}">
